File: _saved_LifxSwitch.sch (KiCad schematic (older format))
At the start: 20 parts

Commit message: something
Parts:
- added R?: 10k, symbol R
Connections:
- net +3V3: now also R?.1
- net at U?.3 (CH_PD): now also R?.2
Changed lines of the file:
@@
 NoConn ~ 6750 3900
 NoConn ~ 6750 4000
+Wire Wire Line
+	10100 3500 10750 3500
+Wire Wire Line
+	10750 3500 10750 3400
+$Comp
+L R R?
+U 1 1 5B2A6DFF
+P 10750 3250
+F 0 "R?" V 10830 3250 50  0000 C CNN
+F 1 "10k" V 10750 3250 50  0000 C CNN
+F 2 "" V 10680 3250 50  0001 C CNN
+F 3 "" H 10750 3250 50  0001 C CNN
+	1    10750 3250
+	1    0    0    -1
+$EndComp
+$Comp
+L VCC #PWR?
+U 1 1 5B2A6E44
+P 10750 3100
+F 0 "#PWR?" H 10750 2950 50  0001 C CNN
+F 1 "VCC" H 10750 3250 50  0000 C CNN
+F 2 "" H 10750 3100 50  0001 C CNN
+F 3 "" H 10750 3100 50  0001 C CNN
+	1    10750 3100
+	1    0    0    -1
+$EndComp
 $EndSCHEMATC
