File: schematic/_saved_LifxSwitch.sch (KiCad schematic (older format))
At the start: 27 parts

Commit message: Completed Schematic
Parts:
- removed C?: 4.7uF, symbol C
- removed J?: Expansion, symbol Conn_01x03
- removed L?: 3.3uH, symbol L
- removed R?: 50k, symbol R
- removed R?: 25k, symbol R
- removed U?: ST1S06, symbol ST1S06
- added C1, C3: 4.7uF, symbol C
- added C2, C4: 0.1uF, symbol C
- added D1: SP0503BAHTG, SOT192P237X122-4N, symbol SP0503BAHTG
- added D2, D3: LED, symbol LED
- added J2: Conn_01x04, symbol Conn_01x04
- added J4: CP2102, symbol Conn_01x02
- added J5: Arcade, symbol Conn_01x01
- added R1: 1k, symbol R
- added R2: 22.1k, symbol R
- added R3: 47.5k, symbol R
- added U2: CP2102N-A01-GQFN20, SILABS_QFN20, symbol CP2102N-A01-GQFN20
- gave numbers to parts that had none: 21
Connections:
- net +3V3: now also R4.1, C1.2, C2.2, D2.2 (A), D3.2 (A), R1.1, U2.6 (VDD)
- net +5V: now also C3.2, C4.2, D1.3 (B), R2.1, U2.7 (VREGIN)
- net Gpio15: now also J2.1 (Pin_1)
- net Gpio2: now also J2.2 (Pin_2)
- net Gpio9: now also J2.4 (Pin_4)
- net LightStatus: now also J5.1 (Pin_1)
- net RX: now also U2.18 (TXD)
- net TX: now also U2.17 (RXD)
- net VSS: now also C7.1, C8.1, J3.5 (Shield), C1.1, C2.1, C3.1, C4.1, D1.1 (GND), R3.2, U2.12 (GND), U2.21 (GND), U2.3 (GND)
- net Gpio0: now reaches U3.8 (RDY), U4.12 (GPIO0)
- net Gpio0: now also J2.3 (Pin_3)
- net at J3.2 (D-): now also D1.2 (A), U2.5 (D)
- net at J3.3 (D+): now also D1.4 (C), U2.4 (D+)
- new net: D2.1 (K), U2.19 (GPIO.3/RXT)
- new net: D3.1 (K), U2.20 (GPIO.2/TXT)
- new net: R2.2, R3.1, U2.8 (VBUS)
- new net: R1.2, U2.9 (RST)
- new net G0: J4.1 (Pin_1), U2.2 (GPIO.0/CLK)
- new net G1: J4.2 (Pin_2), U2.1 (GPIO.1/RS485)
- no-connect marks 2 -> 15
Other:
- moved on the sheet: C5, C6, C7, C8, C9, D4, D5, D6, D7, J3, R10, R4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
