File: schematic/_saved_LifxSwitch.sch (KiCad schematic (older format))
At the start: 36 parts, among them J1 Serial, J2 Expansion, J3 USB_A, J4 CP_Expansion, J5 Arcade, J6 Power, U1 TouchStrip, U2 CP2102N-A01-GQFN20, U3 IQS572, U4 ESP-12E

Commit message: Finished V1 schematic
Parts:
- added C10: 10uF, Capacitors_SMD:C_0805, symbol C
- added C11: 0.1uF, Capacitors_SMD:C_0805, symbol C
Connections:
- net +3V3: now also C10.1, C11.1
- net VSS: now also C10.2, C11.2
Changed lines of the file:
@@
 L VCC #PWR09
 U 1 1 5B29EAF7
-P 10050 3300
-F 0 "#PWR09" H 10050 3150 50  0001 C CNN
-F 1 "VCC" H 10050 3450 50  0000 C CNN
-F 2 "" H 10050 3300 50  0001 C CNN
-F 3 "" H 10050 3300 50  0001 C CNN
-	1    10050 3300
+P 10400 3300
+F 0 "#PWR09" H 10400 3150 50  0001 C CNN
+F 1 "VCC" H 10400 3450 50  0000 C CNN
+F 2 "" H 10400 3300 50  0001 C CNN
+F 3 "" H 10400 3300 50  0001 C CNN
+	1    10400 3300
 	0    1    1    0
 $EndComp
@@
 	0    1    1    0
 $EndComp
+Wire Wire Line
+	10050 3300 10400 3300
+$Comp
+L C C11
+U 1 1 5B35919E
+P 10350 3450
+F 0 "C11" H 10375 3550 50  0000 L CNN
+F 1 "0.1uF" H 10375 3350 50  0000 L CNN
+F 2 "Capacitors_SMD:C_0805" H 10388 3300 50  0001 C CNN
+F 3 "" H 10350 3450 50  0001 C CNN
+	1    10350 3450
+	1    0    0    -1
+$EndComp
+$Comp
+L C C10
+U 1 1 5B359203
+P 10100 3450
+F 0 "C10" H 10125 3550 50  0000 L CNN
+F 1 "10uF" H 10125 3350 50  0000 L CNN
+F 2 "Capacitors_SMD:C_0805" H 10138 3300 50  0001 C CNN
+F 3 "" H 10100 3450 50  0001 C CNN
+	1    10100 3450
+	1    0    0    -1
+$EndComp
+Wire Wire Line
+	10100 3600 10350 3600
+$Comp
+L VSS #PWR026
+U 1 1 5B3595DA
+P 10250 3600
+F 0 "#PWR026" H 10250 3450 50  0001 C CNN
+F 1 "VSS" H 10250 3750 50  0000 C CNN
+F 2 "" H 10250 3600 50  0001 C CNN
+F 3 "" H 10250 3600 50  0001 C CNN
+	1    10250 3600
+	-1   0    0    1
+$EndComp
+Connection ~ 10100 3300
+Connection ~ 10350 3300
+Connection ~ 10250 3600
 $EndSCHEMATC
